Commit message: Add optional Kachaka mobile base to the URDF
Add the use_kachaka_base argument and build the base structure conditionally.
The fixed base keeps the world -> body_base_link joint, while the Kachaka base
builds base_footprint -> Kachaka platform -> vehicle body -> body_base_link and
has no world link.

Include the Kachaka xacro files inside the conditional so the default
configuration still parses when the Kachaka packages are not installed.

Rename the upper body root from base_link to body_base_link, because the
Kachaka platform contributes its own link named base_link and the two would
otherwise collide.

File: urdf/sciurus17.urdf.xacro (robot description, xacro)
@@ -15,4 +15,5 @@
   <xacro:include filename="$(find sciurus17_description)/urdf/sciurus17_gazebo.xacro"/>
   <xacro:include filename="$(find sciurus17_description)/urdf/sciurus17.gazebo_ros2_control.xacro"/>
+  <!-- Arguments: declare before use in conditionals -->
   <xacro:arg name="use_gazebo" default="false" />
   <xacro:arg name="use_gazebo_head_camera" default="false" />
@@ -20,4 +21,16 @@
   <xacro:arg name="use_mock_components" default="false" />
   <xacro:arg name="use_isaacsim" default="false" />
+  <xacro:arg name="use_kachaka_base" default="false" />
+  <!-- Kachaka base support (optional).
+       These are included only when the Kachaka base is requested so that the default
+       fixed-base configuration does not depend on the Kachaka packages being installed. -->
+  <xacro:if value="$(arg use_kachaka_base)">
+    <xacro:include filename="$(find sciurus17_kachaka_description)/urdf/_kachaka_base.urdf.xacro"/>
+    <xacro:include filename="$(find sciurus17_kachaka_description)/urdf/_sciurus17_vehicle_body.urdf.xacro"/>
+    <!-- Kachaka mobile robot (for mobile manipulator mode) -->
+    <xacro:include filename="$(find kachaka_description)/urdf/_values.urdf.xacro"/>
+    <xacro:include filename="$(find kachaka_description)/urdf/_kachaka.urdf.xacro"/>
+    <xacro:include filename="$(find kachaka_description)/urdf/_materials.urdf.xacro"/>
+  </xacro:if>
   <xacro:arg name="port_name" default="/dev/sciurus17spine" />
   <xacro:arg name="baudrate" default="3000000" />
@@ -84,10 +97,42 @@
   <!-- 参照: https://github.com/rt-net/sciurus17_description/pull/6 -->
   <xacro:property name="JOINT_GRIPPER_L_UPPER_LIMIT" value="${radians(0.05)}"/>
-  <!-- Used for fixing robot 'base_link'  to Gazebo 'world' -->
-  <link name="world"/>
-  <joint name="base_link_to_world_joint" type="fixed">
-    <parent link="world"/>
-    <child link="base_link"/>
-  </joint>
+  <!-- Conditional base configuration: with or without Kachaka base -->
+  <xacro:if value="$(arg use_kachaka_base)">
+    <!-- With Kachaka mobile base configuration:
+         base_footprint -> kachaka_robot (mobile platform) -> kachaka_base_link ->
+         sciurus17_vehicle_body -> sciurus17_body
+         base_footprint allows proper mobile manipulation with full Kachaka mobility.
+    -->
+    <link name="base_footprint"/>
+    <xacro:kachaka_robot parent="base_footprint">
+      <origin xyz="0 0 0" rpy="0 0 0"/>
+    </xacro:kachaka_robot>
+    <!-- Kachaka static base frame attached to the mobile base_link -->
+    <xacro:kachaka_base parent="base_link">
+      <origin xyz="0.0 0.0 0.1408" rpy="0.0 0.0 0.0" />
+    </xacro:kachaka_base>
+    <!-- Add vehicle body (structural frame connecting Kachaka to Sciurus17 upper body) -->
+    <xacro:sciurus17_vehicle_body parent="kachaka_base_link">
+      <origin rpy="0 0 0" xyz="${0.007+0.13/2} 0.0 0.0"/>
+    </xacro:sciurus17_vehicle_body>
+    <!-- Connect the upper body to the vehicle body's upper section -->
+    <joint name="base_link_to_world_joint" type="fixed">
+      <parent link="sciurus17_vehicle_body_upper_link"/>
+      <child link="body_base_link"/>
+      <origin xyz="${-0.062+0.13/2+0.02} 0 0.34" rpy="0 0 0"/>
+    </joint>
+  </xacro:if>
+  <xacro:unless value="$(arg use_kachaka_base)">
+    <!-- Used for fixing robot 'body_base_link' to Gazebo 'world' -->
+    <link name="world"/>
+    <!-- Upper body only: world -> body_base_link (standard fixed sciurus17 configuration)
+         This is a fixed manipulator without mobile base.
+    -->
+    <joint name="base_link_to_world_joint" type="fixed">
+      <parent link="world"/>
+      <child link="body_base_link"/>
+      <origin xyz="0 0 0" rpy="0 0 0"/>
+    </joint>
+  </xacro:unless>
   <xacro:sciurus17_body/>
   <xacro:sciurus17_head/>

File: urdf/sciurus17_body.xacro (robot description, xacro)
@@ -2,5 +2,5 @@
 <robot xmlns:xacro="http://ros.org/wiki/xacro">
   <xacro:macro name="sciurus17_body">
-    <link name="base_link">
+    <link name="body_base_link">
       <visual>
         <geometry>
@@ -22,5 +22,5 @@
     </link>
     <joint name="waist_yaw_joint" type="revolute">
-      <parent link="base_link" />
+      <parent link="body_base_link" />
       <child link="body_link" />
       <origin xyz="0.0 0.0 0.1315" rpy="0 0 0"/>

File: urdf/sciurus17_gazebo.xacro (robot description, xacro)
@@ -35,5 +35,5 @@
       </plugin>
     </gazebo>
-    <gazebo reference="base_link">
+    <gazebo reference="body_base_link">
       <xacro:material_gazebo_white/>
     </gazebo>

Commit message: Allow the head, arms and grippers to be left out
Add enable_head, enable_arm_right, enable_arm_left, enable_gripper_right and
enable_gripper_left so the packages can drive a partially assembled robot. Each
defaults to true, so the fully assembled robot is unchanged.

A gripper is only built when its arm is, since it mounts on the arm's wrist.

The head camera color frames are built with the head, because they descend from
head_camera_link and would otherwise reference a link that does not exist.

The arguments are compared as text so that both 'true' and 'True' are accepted.

File: urdf/sciurus17.urdf.xacro (robot description, xacro)
@@ -22,4 +22,21 @@
   <xacro:arg name="use_isaacsim" default="false" />
   <xacro:arg name="use_kachaka_base" default="false" />
+  <!-- Activate components.
+       A gripper can only be built when its arm is, since it mounts on the arm's
+       last link. Requesting a gripper without its arm therefore has no effect. -->
+  <xacro:arg name="enable_head" default="true" />
+  <xacro:arg name="enable_arm_right" default="true" />
+  <xacro:arg name="enable_arm_left" default="true" />
+  <xacro:arg name="enable_gripper_right" default="true" />
+  <xacro:arg name="enable_gripper_left" default="true" />
+  <!-- Compared as text so that both 'true' and 'True' are accepted, matching the
+       spelling used by the other arguments of this file. -->
+  <xacro:property name="ENABLE_HEAD" value="${'$(arg enable_head)'.lower() == 'true'}"/>
+  <xacro:property name="ENABLE_ARM_R" value="${'$(arg enable_arm_right)'.lower() == 'true'}"/>
+  <xacro:property name="ENABLE_ARM_L" value="${'$(arg enable_arm_left)'.lower() == 'true'}"/>
+  <xacro:property name="ENABLE_GRIPPER_R"
+    value="${'$(arg enable_gripper_right)'.lower() == 'true' and ENABLE_ARM_R}"/>
+  <xacro:property name="ENABLE_GRIPPER_L"
+    value="${'$(arg enable_gripper_left)'.lower() == 'true' and ENABLE_ARM_L}"/>
   <!-- Kachaka base support (optional).
        These are included only when the Kachaka base is requested so that the default
@@ -136,9 +153,21 @@
   </xacro:unless>
   <xacro:sciurus17_body/>
-  <xacro:sciurus17_head/>
-  <xacro:sciurus17_right_arm/>
-  <xacro:sciurus17_right_gripper/>
-  <xacro:sciurus17_left_arm/>
-  <xacro:sciurus17_left_gripper/>
+  <xacro:if value="${ENABLE_HEAD}">
+    <xacro:sciurus17_head/>
+  </xacro:if>
+  <xacro:if value="${ENABLE_ARM_R}">
+    <xacro:sciurus17_right_arm/>
+    <xacro:sciurus17_right_wrist/>
+  </xacro:if>
+  <xacro:if value="${ENABLE_GRIPPER_R}">
+    <xacro:sciurus17_right_gripper/>
+  </xacro:if>
+  <xacro:if value="${ENABLE_ARM_L}">
+    <xacro:sciurus17_left_arm/>
+    <xacro:sciurus17_left_wrist/>
+  </xacro:if>
+  <xacro:if value="${ENABLE_GRIPPER_L}">
+    <xacro:sciurus17_left_gripper/>
+  </xacro:if>
   <xacro:unless value="$(arg use_gazebo)">
     <xacro:sciurus17_ros2_control_settings
@@ -158,5 +187,6 @@
     <xacro:sciurus17_gazebo_ros2_control_settings/>
   </xacro:if>
-  <xacro:if value="${'$(arg use_gazebo)' == 'true' or '$(arg use_isaacsim)' == 'true'}">
+  <!-- These frames hang off head_camera_link, so they only exist with the head. -->
+  <xacro:if value="${('$(arg use_gazebo)' == 'true' or '$(arg use_isaacsim)' == 'true') and ENABLE_HEAD}">
     <joint name="head_camera_color_joint" type="fixed">
       <origin xyz="0 0.015 0" rpy="0 0 0" />
