Commit message: Move the wrist link out of the gripper macros
r_link7 and l_link7 are the child links of the arms' last joints, not part of
the gripper, but they were defined inside the gripper macros. Building an arm
without its gripper therefore produced a URDF whose last arm joint referenced a
missing child link.

Give each wrist its own macro so the arm can supply it independently.

File: urdf/sciurus17_left_gripper.xacro (robot description, xacro)
@@ -1,5 +1,7 @@
 <?xml version="1.0"?>
 <robot xmlns:xacro="http://ros.org/wiki/xacro">
-  <xacro:macro name="sciurus17_left_gripper">
+  <!-- The wrist link is part of the arm: it is the child of X_arm_joint7 and must
+       exist even when the gripper is not built. -->
+  <xacro:macro name="sciurus17_left_wrist">
     <link name="l_link7">
       <visual>
@@ -22,4 +24,6 @@
       </inertial>
     </link>
+  </xacro:macro>
+  <xacro:macro name="sciurus17_left_gripper">
     <joint name="l_gripper_joint" type="revolute">
       <parent link="l_link7" />

File: urdf/sciurus17_right_gripper.xacro (robot description, xacro)
@@ -1,5 +1,7 @@
 <?xml version="1.0"?>
 <robot xmlns:xacro="http://ros.org/wiki/xacro">
-  <xacro:macro name="sciurus17_right_gripper">
+  <!-- The wrist link is part of the arm: it is the child of X_arm_joint7 and must
+       exist even when the gripper is not built. -->
+  <xacro:macro name="sciurus17_right_wrist">
     <link name="r_link7">
       <visual>
@@ -22,4 +24,6 @@
       </inertial>
     </link>
+  </xacro:macro>
+  <xacro:macro name="sciurus17_right_gripper">
     <joint name="r_gripper_joint" type="revolute">
       <parent link="r_link7" />
